File: SparkFun_I2S_Audio_Breakout.brd (EAGLE design)
At the start: 20.3 x 20.3 mm, 39 parts, among them IC1 MAX98375A

Commit message: Fixed IC1 Value
-Fixed IC1 value from MAX98375A to MAX98357A
Parts:
- added FRAME1: FRAME-LETTER, SparkFun-Aesthetics:CREATIVE_COMMONS
- IC1: value MAX98375A -> MAX98357A
Other:
- board text added: "Alex Wende"
- board text added: "Units: Inches"
Changed lines of the file:
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@@
 <?xml version="1.0" encoding="utf-8"?>
 <!DOCTYPE eagle SYSTEM "eagle.dtd">
-<eagle version="9.1.0">
+<eagle version="9.1.1">
 <drawing>
 <settings>
@@
 <setting verticaltext="up"/>
 </settings>
-<grid distance="0.05" unitdist="inch" unit="inch" style="lines" multiple="1" display="yes" altdistance="0.005" altunitdist="inch" altunit="inch"/>
+<grid distance="50" unitdist="mil" unit="inch" style="lines" multiple="1" display="yes" altdistance="0.005" altunitdist="inch" altunit="inch"/>
 <layers>
 <layer number="1" name="Top" color="4" fill="1" visible="yes" active="yes"/>
@@
 <layer number="23" name="tOrigins" color="15" fill="1" visible="yes" active="yes"/>
 <layer number="24" name="bOrigins" color="15" fill="1" visible="yes" active="yes"/>
-<layer number="25" name="tNames" color="7" fill="1" visible="yes" active="yes"/>
-<layer number="26" name="bNames" color="7" fill="1" visible="yes" active="yes"/>
-<layer number="27" name="tValues" color="7" fill="1" visible="yes" active="yes"/>
-<layer number="28" name="bValues" color="7" fill="1" visible="yes" active="yes"/>
+<layer number="25" name="tNames" color="7" fill="1" visible="no" active="yes"/>
+<layer number="26" name="bNames" color="7" fill="1" visible="no" active="yes"/>
+<layer number="27" name="tValues" color="7" fill="1" visible="no" active="yes"/>
+<layer number="28" name="bValues" color="7" fill="1" visible="no" active="yes"/>
 <layer number="29" name="tStop" color="7" fill="3" visible="yes" active="yes"/>
-<layer number="30" name="bStop" color="7" fill="6" visible="yes" active="yes"/>
-<layer number="31" name="tCream" color="7" fill="4" visible="yes" active="yes"/>
-<layer number="32" name="bCream" color="7" fill="5" visible="yes" active="yes"/>
-<layer number="33" name="tFinish" color="6" fill="3" visible="yes" active="yes"/>
-<layer number="34" name="bFinish" color="6" fill="6" visible="yes" active="yes"/>
-<layer number="35" name="tGlue" color="7" fill="4" visible="yes" active="yes"/>
-<layer number="36" name="bGlue" color="7" fill="5" visible="yes" active="yes"/>
-<layer number="37" name="tTest" color="7" fill="1" visible="yes" active="yes"/>
-<layer number="38" name="bTest" color="7" fill="1" visible="yes" active="yes"/>
+<layer number="30" name="bStop" color="7" fill="6" visible="no" active="yes"/>
+<layer number="31" name="tCream" color="7" fill="4" visible="no" active="yes"/>
+<layer number="32" name="bCream" color="7" fill="5" visible="no" active="yes"/>
+<layer number="33" name="tFinish" color="6" fill="3" visible="no" active="yes"/>
+<layer number="34" name="bFinish" color="6" fill="6" visible="no" active="yes"/>
+<layer number="35" name="tGlue" color="7" fill="4" visible="no" active="yes"/>
+<layer number="36" name="bGlue" color="7" fill="5" visible="no" active="yes"/>
+<layer number="37" name="tTest" color="7" fill="1" visible="no" active="yes"/>
+<layer number="38" name="bTest" color="7" fill="1" visible="no" active="yes"/>
 <layer number="39" name="tKeepout" color="4" fill="11" visible="yes" active="yes"/>
 <layer number="40" name="bKeepout" color="1" fill="11" visible="yes" active="yes"/>
@@
 <layer number="42" name="bRestrict" color="1" fill="10" visible="yes" active="yes"/>
 <layer number="43" name="vRestrict" color="2" fill="10" visible="yes" active="yes"/>
-<layer number="44" name="Drills" color="7" fill="1" visible="yes" active="yes"/>
-<layer number="45" name="Holes" color="7" fill="1" visible="yes" active="yes"/>
-<layer number="46" name="Milling" color="3" fill="1" visible="yes" active="yes"/>
-<layer number="47" name="Measures" color="7" fill="1" visible="yes" active="yes"/>
+<layer number="44" name="Drills" color="7" fill="1" visible="no" active="yes"/>
+<layer number="45" name="Holes" color="7" fill="1" visible="no" active="yes"/>
+<layer number="46" name="Milling" color="3" fill="1" visible="no" active="yes"/>
+<layer number="47" name="Measures" color="7" fill="1" visible="no" active="yes"/>
 <layer number="48" name="Document" color="7" fill="1" visible="yes" active="yes"/>
 <layer number="49" name="Reference" color="7" fill="1" visible="yes" active="yes"/>
@@
 <wire x1="9.017" y1="9.44118125" x2="9.271" y2="9.44118125" width="0.2032" layer="41"/>
 <text x="13.97" y="0.3175" size="1.016" layer="16" font="vector" ratio="20" rot="SR0" align="bottom-center">v10</text>
+<text x="12.7635" y="-18.288" size="2.1844" layer="51" font="vector" ratio="15" align="center-left">Alex Wende</text>
+<dimension x1="0" y1="1.27" x2="20.32" y2="1.27" x3="10.16" y3="-5.08" textsize="1.27" textratio="15" layer="47" unit="inch"/>
+<dimension x1="1.27" y1="0" x2="1.27" y2="20.32" x3="-5.08" y3="10.16" textsize="1.27" textratio="15" layer="47" unit="inch"/>
+<dimension x1="0" y1="1.27" x2="1.27" y2="1.27" x3="0.635" y3="-2.54" textsize="1.27" textratio="15" layer="47" unit="inch"/>
+<dimension x1="17.145" y1="3.175" x2="20.32" y2="3.175" x3="18.7325" y3="-2.54" textsize="1.27" textratio="15" layer="47" unit="inch" precision="3"/>
+<dimension x1="17.145" y1="17.145" x2="20.32" y2="17.145" x3="18.7325" y3="22.86" textsize="1.27" textratio="15" layer="47" unit="inch" precision="3"/>
+<dimension x1="17.145" y1="17.145" x2="17.145" y2="20.32" x3="29.21" y3="18.7325" textsize="1.27" textratio="15" layer="47" unit="inch" precision="3"/>
+<dimension x1="17.145" y1="3.175" x2="17.145" y2="0" x3="29.21" y3="1.5875" textsize="1.27" textratio="15" layer="47" unit="inch" precision="3"/>
+<dimension x1="1.27" y1="19.05" x2="0.338125" y2="19.912846875" x3="-5.3852125" y3="25.212228125" textsize="1.27" textratio="15" layer="47" dtype="radius" unit="inch" precision="3"/>
+<text x="5.08" y="-6.35" size="1.27" layer="47" font="vector" ratio="15" align="center-left">Units: Inches</text>
+<dimension x1="1.27" y1="2.54" x2="1.27" y2="0" x3="-2.54" y3="1.27" textsize="1.27" textratio="15" layer="47" unit="inch" precision="3"/>
 <text x="18.415" y="4.826" size="1.778" layer="21" font="vector" ratio="15">+</text>
 <text x="19.812" y="13.843" size="1.778" layer="21" font="vector" ratio="15" rot="R90">-</text>
@@
 <attribute name="PROD_ID" value="CAP-00810" x="9.6266" y="5.0292" size="1.778" layer="27" rot="R270" display="off"/>
 </element>
-<element name="IC1" library="SparkFun-IC-Amplifiers" package="TQFN-16" value="MAX98375A" x="9.144" y="10.16" rot="R270">
+<element name="IC1" library="SparkFun-IC-Amplifiers" package="TQFN-16" value="MAX98357A" x="9.144" y="10.16" rot="R270">
 <attribute name="PROD_ID" value="IC-14032" x="9.144" y="10.16" size="1.778" layer="27" rot="R270" display="off"/>
 </element>
@@
 <element name="FD1" library="SparkFun-Aesthetics" package="FIDUCIAL-MICRO" value="FIDUCIALUFIDUCIAL" x="19.4818" y="0.8128"/>
 <element name="FD2" library="SparkFun-Aesthetics" package="FIDUCIAL-MICRO" value="FIDUCIALUFIDUCIAL" x="0.8128" y="19.4818"/>
+<element name="FRAME1" library="SparkFun-Aesthetics" package="CREATIVE_COMMONS" value="FRAME-LETTER" x="-13.97" y="-19.05"/>
 <element name="LOGO1" library="SparkFun-Aesthetics" package="SFE_LOGO_NAME_FLAME_.1" value="SFE_LOGO_NAME_FLAME.1_INCH" x="16.891" y="16.129" rot="SMR270"/>
 <element name="LOGO2" library="SparkFun-Aesthetics" package="OSHW-LOGO-S" value="OSHW-LOGOS" x="12.573" y="13.462" rot="MR270"/>
